Commit message: Full work

File: description/robot.urdf.xacro (robot description, xacro)
@@ -2,3 +2,4 @@
 <robot xmlns:xacro="http://www.ros.org/wiki/xacro"  name="robot">
    <xacro:include filename="robot_core.xacro" />
+   <xacro:include filename="gazebo_control.xacro"/>
 </robot>

File: description/robot_core.xacro (robot description, xacro)
@@ -39,4 +39,7 @@
         </xacro:inertial_box>
     </link>
+    <gazebo reference="chassis">
+        <material>Gazebo/White</material>
+    </gazebo>
     <!-- LEFT WHEEL -->
 <joint name="left_wheel_joint" type="continuous">
@@ -62,4 +65,7 @@
     </xacro:inertial_cylinder>
 </link>
+<gazebo reference="left_wheel">
+    <material>Gazebo/Blue</material>
+</gazebo>
 <!-- RIGHT WHEEL -->
 <joint name="right_wheel_joint" type="continuous">
@@ -85,4 +91,7 @@
     </xacro:inertial_cylinder>
 </link>
+<gazebo reference="right_wheel">
+    <material>Gazebo/Blue</material>
+</gazebo>
 <!-- CASTER WHEEL -->
 <joint name="caster_wheel_joint" type="fixed">
@@ -107,3 +116,8 @@
     </xacro:inertial_sphere>
 </link>
+<gazebo reference="caster_wheel">
+    <material>Gazebo/Black</material>
+    <mu1 value="0.001"/>
+    <mu2 value="0.001"/>
+</gazebo>
 </robot>
